File: files/2017-04-14-relai-bistable-commande-tension/kicad/relai-bistable-commande-tension.sch (KiCad schematic (older format))
At the start: 17 parts, among them T1 BC337, T2 BC337

Commit message: schéma électrique pour relai bistable
Parts:
- added A?: ALIMENTATION-IRM-03-3.3, symbol ALIMENTATION-IRM-03-3.3
- R5, R6: value 10kΩ -> 1kΩ
Connections:
- wire segments 56 -> 60
Other:
- moved on the sheet: A1, C1, D1, D2, J1, J2, J3, OC1, R1, R2, R3, R4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

Commit message: modif kicad
Parts:
- removed A?: ALIMENTATION-IRM-03-3.3, symbol ALIMENTATION-IRM-03-3.3
- added ALIM1: ALIMENTATION-IRM-03-3.3, symbol ALIMENTATION-IRM-03-3.3
- C1: footprint (none) -> Capacitors_THT:CP_Radial_D5.0mm_P2.50mm
- D1, D2: footprint (none) -> Diodes_THT:D_DO-41_SOD81_P7.62mm_Horizontal
- J1, J2: footprint (none) -> Connectors_Phoenix:PhoenixContact_MC-G_03x3.50mm_Angled
- J3: footprint (none) -> Connectors_Phoenix:PhoenixContact_MC-G_02x3.50mm_Angled
- OC1: footprint (none) -> empreintes:Optocoupleur_SFH620
- R1: renamed from R3; footprint (none) -> Resistors_THT:Resistor_Horizontal_RM7mm
- R2: renamed from R4; footprint (none) -> Resistors_THT:Resistor_Horizontal_RM7mm
- R3: renamed from R1; footprint (none) -> Resistors_THT:Resistor_Horizontal_RM7mm
- R4: renamed from R2; footprint (none) -> Resistors_THT:Resistor_Horizontal_RM7mm
- R5, R6: footprint (none) -> Resistors_THT:Resistor_Horizontal_RM7mm
- RB1: footprint (none) -> empreintes:Relai_Bistable_Panasonic_ADW1203W
- T1: renamed from T2; footprint TO-92 -> TO_SOT_Packages_THT:TO-92_Inline_Narrow_Oval
- T2: renamed from T1; footprint TO-92 -> TO_SOT_Packages_THT:TO-92_Inline_Narrow_Oval
- renumbered A1 to APM1
Connections:
- net labels added: AC, Earth
- wire segments 60 -> 55
Other:
- moved on the sheet: APM1, C1, D1, D2, J1, J2, J3, OC1, R1, R2, R3, R4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

Commit message: update kicad
Parts:
- removed ALIM1: ALIMENTATION-IRM-03-3.3, symbol ALIMENTATION-IRM-03-3.3
- added ALIM1: ALIM-IRM-03-3.3, empreintes:AC-DC_power_supply_IRM-03, symbol ALIM-IRM-03-3.3
- added R0: 1.5Ω, Resistors_THT:Resistor_Horizontal_RM7mm, symbol R
- APM1: footprint (none) -> empreintes:Arduino_Pro_Mini
- J1, J2: footprint Connectors_Phoenix:PhoenixContact_MC-G_03x3.50mm_Angled -> Connectors_Phoenix:PhoenixContact_MC-G_03x5.08mm_Angled
- J3: footprint Connectors_Phoenix:PhoenixContact_MC-G_02x3.50mm_Angled -> Connectors_Phoenix:PhoenixContact_MC-G_02x5.08mm_Angled
Connections:
- wire segments 55 -> 57
- no-connect marks 0 -> 19
Other:
- moved on the sheet: R5

Commit message: modif PCB Kicad
Other:
- moved on the sheet: APM1
Changed lines of the file:
@@
 L ARDUINO-PRO-MINI APM1
 U 1 1 58F25AB8
-P 3900 2050
-F 0 "APM1" H 3900 500 60  0000 C CNN
-F 1 "ARDUINO-PRO-MINI" V 3900 1200 60  0000 C CNN
-F 2 "empreintes:Arduino_Pro_Mini" H 3900 2050 60  0001 C CNN
-F 3 "" H 3900 2050 60  0001 C CNN
-	1    3900 2050
+P 3900 1850
+F 0 "APM1" H 3900 300 60  0000 C CNN
+F 1 "ARDUINO-PRO-MINI" V 3900 1000 60  0000 C CNN
+F 2 "empreintes:Arduino_Pro_Mini" H 3900 1850 60  0001 C CNN
+F 3 "" H 3900 1850 60  0001 C CNN
+	1    3900 1850
 	0    1    -1   0
 $EndComp
@@
 L GND #PWR05
 U 1 1 58F26E0D
-P 3500 1300
-F 0 "#PWR05" H 3500 1050 50  0001 C CNN
-F 1 "GND" H 3500 1150 50  0000 C CNN
-F 2 "" H 3500 1300 50  0000 C CNN
-F 3 "" H 3500 1300 50  0000 C CNN
-	1    3500 1300
+P 3500 1100
+F 0 "#PWR05" H 3500 850 50  0001 C CNN
+F 1 "GND" H 3500 950 50  0000 C CNN
+F 2 "" H 3500 1100 50  0000 C CNN
+F 3 "" H 3500 1100 50  0000 C CNN
+	1    3500 1100
 	-1   0    0    1
 $EndComp
@@
 L +3.3V #PWR06
 U 1 1 58F26E82
-P 3200 1300
-F 0 "#PWR06" H 3200 1150 50  0001 C CNN
-F 1 "+3.3V" H 3200 1440 50  0000 C CNN
-F 2 "" H 3200 1300 50  0000 C CNN
-F 3 "" H 3200 1300 50  0000 C CNN
-	1    3200 1300
+P 3200 1100
+F 0 "#PWR06" H 3200 950 50  0001 C CNN
+F 1 "+3.3V" H 3200 1240 50  0000 C CNN
+F 2 "" H 3200 1100 50  0000 C CNN
+F 3 "" H 3200 1100 50  0000 C CNN
+	1    3200 1100
 	1    0    0    -1
 $EndComp
@@
 	1    0    0    -1
 $EndComp
-NoConn ~ 2500 1500
-NoConn ~ 2600 1500
-NoConn ~ 2700 1500
-NoConn ~ 2800 1500
-NoConn ~ 2900 1500
-NoConn ~ 3000 1500
-NoConn ~ 3100 1500
-NoConn ~ 3200 1500
-NoConn ~ 3400 1500
-NoConn ~ 3600 1500
-NoConn ~ 3600 2600
-NoConn ~ 3500 2600
-NoConn ~ 3400 2600
-NoConn ~ 3300 2600
-NoConn ~ 3100 2600
-NoConn ~ 3000 2600
-NoConn ~ 2900 2600
-NoConn ~ 2800 2600
-NoConn ~ 2700 2600
+NoConn ~ 2500 1300
+NoConn ~ 2600 1300
+NoConn ~ 2700 1300
+NoConn ~ 2800 1300
+NoConn ~ 2900 1300
+NoConn ~ 3000 1300
+NoConn ~ 3100 1300
+NoConn ~ 3200 1300
+NoConn ~ 3400 1300
+NoConn ~ 3600 1300
+NoConn ~ 3600 2400
+NoConn ~ 3500 2400
+NoConn ~ 3400 2400
+NoConn ~ 3100 2400
+NoConn ~ 3000 2400
+NoConn ~ 2800 2400
+NoConn ~ 2700 2400
 $Comp
 L ALIM-IRM-03-3.3 ALIM1
@@
 	2500 2850 2050 2850
 Wire Wire Line
-	3200 2600 3200 2750
-Wire Wire Line
 	4400 2750 4400 2950
 Wire Wire Line
 	4150 2850 2600 2850
 Wire Wire Line
-	2600 2850 2600 2600
-Wire Wire Line
-	2500 2850 2500 2600
-Wire Wire Line
-	3500 1500 3500 1300
-Wire Wire Line
-	3300 1500 3300 1350
-Wire Wire Line
-	3300 1350 3200 1350
-Wire Wire Line
-	3200 1350 3200 1300
+	3500 1300 3500 1100
+Wire Wire Line
+	3300 1300 3300 1150
+Wire Wire Line
+	3300 1150 3200 1150
+Wire Wire Line
+	3200 1150 3200 1100
 Wire Wire Line
 	4200 3700 4200 3750
@@
 Wire Wire Line
 	2650 5450 2650 5200
+NoConn ~ 2900 2400
+Wire Wire Line
+	2500 2850 2500 2400
+Wire Wire Line
+	2600 2850 2600 2400
+Wire Wire Line
+	3200 2400 3200 2750
+NoConn ~ 3300 2400
 $EndSCHEMATC

Commit message: pcb kicad
Parts:
- removed RB1: RELAI-BISTABLE, empreintes:Relai_Bistable_Panasonic_ADW1203W, symbol RELAI-BISTABLE
- added RB1: RELAI-BISTABLE, empreintes:Relai_Bistable_Panasonic_ADW1203W, symbol RELAI-BISTABLE-RESCUE-relai-bistable-commande-tension
Connections:
- net AC: now also J1.1, RB1.3; no longer J1.3
- net Earth: now also J1.3, J2.1; no longer J1.1, J2.3
- net at D2.2 (A), T1.1 (C): now also RB1.-1
- net at D1.1 (K), D2.1 (K), R0.2: now also RB1.+7
- net at D1.2 (A), T2.1 (C): now also RB1.-6
- net at J3.2: now also OC1.2; no longer OC1.1
- net at R5.2: now also OC1.1; no longer OC1.2
- new net: J2.3, RB1.5
Other:
- moved on the sheet: R5
Changed lines of the file:
@@
 EESchema Schematic File Version 2
+LIBS:relai-bistable-commande-tension-rescue
 LIBS:power
 LIBS:device
@@
 $EndComp
 $Comp
-L ARDUINO-PRO-MINI APM1
-U 1 1 58F25AB8
-P 3900 1850
-F 0 "APM1" H 3900 300 60  0000 C CNN
-F 1 "ARDUINO-PRO-MINI" V 3900 1000 60  0000 C CNN
-F 2 "empreintes:Arduino_Pro_Mini" H 3900 1850 60  0001 C CNN
-F 3 "" H 3900 1850 60  0001 C CNN
-	1    3900 1850
-	0    1    -1   0
-$EndComp
-$Comp
-L RELAI-BISTABLE RB1
-U 1 1 58F25BD3
-P 3100 4850
-F 0 "RB1" H 3100 5050 60  0000 C CNN
-F 1 "RELAI-BISTABLE" H 3100 4950 60  0000 C CNN
-F 2 "empreintes:Relai_Bistable_Panasonic_ADW1203W" H 3100 4850 60  0001 C CNN
-F 3 "" H 3100 4850 60  0001 C CNN
-	1    3100 4850
-	-1   0    0    1
-$EndComp
-$Comp
 L D D1
 U 1 1 58F26031
@@
 F 3 "" H 3525 5750 50  0001 C CNN
 	1    3550 5650
-	0    1    -1   0
+	0    -1   -1   0
 $EndComp
 $Comp
@@
 F 3 "" H 2625 5750 50  0001 C CNN
 	1    2650 5650
-	0    1    -1   0
+	0    -1   -1   0
 $EndComp
 $Comp
@@
 U 1 1 58F28418
 P 4450 5650
-F 0 "J3" V 4450 5400 50  0000 C TNN
+F 0 "J3" V 4450 5900 50  0000 C TNN
 F 1 "~" V 4300 5650 50  0000 C TNN
 F 2 "Connectors_Phoenix:PhoenixContact_MC-G_02x5.08mm_Angled" H 4450 5425 50  0001 C CNN
 F 3 "" H 4425 5650 50  0001 C CNN
 	1    4450 5650
-	0    1    -1   0
+	0    -1   -1   0
 $EndComp
 $Comp
 L R R5
 U 1 1 58F2940D
-P 4550 5200
-F 0 "R5" V 4450 5200 50  0000 C CNN
-F 1 "1kΩ" V 4650 5200 50  0000 C CNN
-F 2 "Resistors_THT:Resistor_Horizontal_RM7mm" V 4480 5200 50  0001 C CNN
-F 3 "" H 4550 5200 50  0000 C CNN
-	1    4550 5200
+P 4350 5200
+F 0 "R5" V 4250 5200 50  0000 C CNN
+F 1 "1kΩ" V 4450 5200 50  0000 C CNN
+F 2 "Resistors_THT:Resistor_Horizontal_RM7mm" V 4280 5200 50  0001 C CNN
+F 3 "" H 4350 5200 50  0000 C CNN
+	1    4350 5200
 	-1   0    0    1
 $EndComp
@@
 	1    1250 3900
 	1    0    0    -1
-$EndComp
-$Comp
-L OPTOCOUPLEUR-SFH620A OC1
-U 1 1 58F28B34
-P 4300 4600
-F 0 "OC1" V 4300 4700 60  0000 C CNN
-F 1 "~" H 4300 4700 60  0000 C CNN
-F 2 "empreintes:Optocoupleur_SFH620" H 4400 4600 60  0001 C CNN
-F 3 "" H 4400 4600 60  0001 C CNN
-	1    4300 4600
-	0    -1   -1   0
 $EndComp
 $Comp
@@
 NoConn ~ 2700 2400
 $Comp
-L ALIM-IRM-03-3.3 ALIM1
-U 1 1 58F5DF1E
-P 1400 4200
-F 0 "ALIM1" H 1400 4000 60  0000 C CNN
-F 1 "ALIM-IRM-03-3.3" H 1450 3800 60  0000 C CNN
-F 2 "empreintes:AC-DC_power_supply_IRM-03" H 1400 4200 60  0001 C CNN
-F 3 "" H 1400 4200 60  0001 C CNN
-	1    1400 4200
-	-1   0    0    -1
-$EndComp
-$Comp
 L R R0
 U 1 1 58F610DE
@@
 	3750 4700 3650 4700
 Wire Wire Line
-	4550 4950 4500 4950
-Wire Wire Line
-	4400 4950 4350 4950
-Wire Wire Line
 	2500 2850 2050 2850
 Wire Wire Line
@@
 Wire Wire Line
 	3100 3550 3100 3500
-Wire Wire Line
-	4550 4950 4550 5050
-Wire Wire Line
-	4550 5350 4550 5450
-Wire Wire Line
-	4350 4950 4350 5450
 Connection ~ 2450 5800
 Wire Wire Line
@@
 	3200 2400 3200 2750
 NoConn ~ 3300 2400
+$Comp
+L ALIM-IRM-03-3.3 ALIM1
+U 1 1 58F76FA5
+P 1400 4200
+F 0 "ALIM1" H 1400 4000 60  0000 C CNN
+F 1 "ALIM-IRM-03-3.3" H 1450 3800 60  0000 C CNN
+F 2 "empreintes:AC-DC_power_supply_IRM-03" H 1400 4200 60  0001 C CNN
+F 3 "" H 1400 4200 60  0001 C CNN
+	1    1400 4200
+	-1   0    0    -1
+$EndComp
+$Comp
+L OPTOCOUPLEUR-SFH620A OC1
+U 1 1 58F77240
+P 4300 4600
+F 0 "OC1" V 4300 4700 60  0000 C CNN
+F 1 "~" H 4300 4700 60  0000 C CNN
+F 2 "empreintes:Optocoupleur_SFH620" H 4400 4600 60  0001 C CNN
+F 3 "" H 4400 4600 60  0001 C CNN
+	1    4300 4600
+	0    -1   -1   0
+$EndComp
+$Comp
+L RELAI-BISTABLE-RESCUE-relai-bistable-commande-tension RB1
+U 1 1 58F772B1
+P 3100 4850
+F 0 "RB1" H 3100 5050 60  0000 C CNN
+F 1 "RELAI-BISTABLE" H 3100 4950 60  0000 C CNN
+F 2 "empreintes:Relai_Bistable_Panasonic_ADW1203W" H 3100 4850 60  0001 C CNN
+F 3 "" H 3100 4850 60  0001 C CNN
+	1    3100 4850
+	-1   0    0    1
+$EndComp
+$Comp
+L ARDUINO-PRO-MINI APM1
+U 1 1 58F77B8D
+P 3900 1850
+F 0 "APM1" H 3900 300 60  0000 C CNN
+F 1 "ARDUINO-PRO-MINI" V 3900 1000 60  0000 C CNN
+F 2 "empreintes:Arduino_Pro_Mini" H 3900 1850 60  0001 C CNN
+F 3 "" H 3900 1850 60  0001 C CNN
+	1    3900 1850
+	0    1    -1   0
+$EndComp
+Wire Wire Line
+	4350 5450 4350 5350
+Wire Wire Line
+	4350 5050 4350 4950
+Wire Wire Line
+	4350 4950 4400 4950
+Wire Wire Line
+	4500 4950 4550 4950
+Wire Wire Line
+	4550 4950 4550 5450
 $EndSCHEMATC

Commit message: plan de masse PCB
Parts:
- removed RB1: RELAI-BISTABLE, empreintes:Relai_Bistable_Panasonic_ADW1203W, symbol RELAI-BISTABLE-RESCUE-relai-bistable-commande-tension
- added RB1: RELAI-BISTABLE, symbol RELAI-BISTABLE
- renumbered D2 to D1, D1 to D2
Connections:
- net AC: now also RB1.5
- net at D1.2 (A), T1.1 (C): now also RB1.-1
- net at D1.1 (K), D2.1 (K), R0.2: now also RB1.+7
- net at D2.2 (A), T2.1 (C): now also RB1.-6
- net at J2.3: now also RB1.3
Changed lines of the file:
@@
 $EndComp
 $Comp
-L D D2
+L D D1
 U 1 1 58F21469
 P 3250 3900
-F 0 "D2" H 3250 3800 50  0000 C CNN
+F 0 "D1" H 3250 3800 50  0000 C CNN
 F 1 "~" H 3250 3800 50  0000 C CNN
 F 2 "Diodes_THT:D_DO-41_SOD81_P7.62mm_Horizontal" H 3250 3900 50  0001 C CNN
@@
 $EndComp
 $Comp
-L D D1
+L D D2
 U 1 1 58F26031
 P 2950 3900
-F 0 "D1" H 2950 3800 50  0000 C CNN
+F 0 "D2" H 2950 3800 50  0000 C CNN
 F 1 "~" H 2950 3800 50  0000 C CNN
 F 2 "Diodes_THT:D_DO-41_SOD81_P7.62mm_Horizontal" H 2950 3900 50  0001 C CNN
@@
 $EndComp
 $Comp
-L RELAI-BISTABLE-RESCUE-relai-bistable-commande-tension RB1
-U 1 1 58F772B1
-P 3100 4850
-F 0 "RB1" H 3100 5050 60  0000 C CNN
-F 1 "RELAI-BISTABLE" H 3100 4950 60  0000 C CNN
-F 2 "empreintes:Relai_Bistable_Panasonic_ADW1203W" H 3100 4850 60  0001 C CNN
-F 3 "" H 3100 4850 60  0001 C CNN
-	1    3100 4850
-	-1   0    0    1
-$EndComp
-$Comp
 L ARDUINO-PRO-MINI APM1
 U 1 1 58F77B8D
@@
 Wire Wire Line
 	4550 4950 4550 5450
+$Comp
+L RELAI-BISTABLE RB1
+U 1 1 58F7CACC
+P 3100 4850
+F 0 "RB1" H 3100 5050 60  0000 C CNN
+F 1 "RELAI-BISTABLE" H 3100 4950 60  0000 C CNN
+F 2 "" H 3100 4850 60  0001 C CNN
+F 3 "" H 3100 4850 60  0001 C CNN
+	1    3100 4850
+	-1   0    0    1
+$EndComp
 $EndSCHEMATC
